File: LD1/Board/LD1-001.brd (EAGLE design)
At the start: 72 x 72 mm, 18 parts, among them IC1 TLC5941NT, IC2 TLC5941NT, IC3 TLC5941NT, IC4 TLC5941NT

Commit message: Updated LD1.
Parts:
- moved C2 2.54 mm to (15.2, 30.5)
- moved C3 2.54 mm to (35.6, 30.5)
- moved C4 2.54 mm to (55.9, 30.5)
- moved IC2 2.54 mm to (19.1, 52.1)
- moved IC3 2.54 mm to (39.4, 52.1)
- moved IC4 2.54 mm to (59.7, 52.1)
- moved JP2 2.54 mm to (8.89, 49.5)
- moved JP3 2.54 mm to (29.2, 49.5)
- moved JP4 2.54 mm to (49.5, 49.5)
- moved R2 2.54 mm to (21.6, 30.5)
- moved R3 2.54 mm to (41.9, 30.5)
- moved R4 2.54 mm to (62.2, 30.5)
- moved CN1 2.00 mm to (6.00, 17.0)
Connections:
- new net N$75: CN1.9, IC1.27, IC2.27, IC3.27, IC4.27
- net GND: no longer IC1.27, IC2.27, IC3.27, IC4.27
Routing:
- net N$75: track 0.00 -> 145.0 mm, vias 0 -> 1
- net BLANK: track 121.6 -> 144.5 mm
- net N$73: track 271.1 -> 293.3 mm
- net XLAT: track 134.8 -> 118.1 mm
- net GND: track 188.1 -> 179.0 mm, vias 1 -> 2
- net N$2: track 62.2 -> 54.4 mm
- net VCC: track 168.8 -> 171.5 mm, vias 0 -> 2
- net N$39: track 8.69 -> 10.7 mm
- net N$47: track 20.3 -> 18.8 mm
- net SCLCK: track 152.7 -> 151.3 mm, vias 0 -> 1
- net N$55: track 18.3 -> 17.3 mm
- net N$1: track 17.7 -> 18.7 mm
- net GSCLCK: track 127.2 -> 126.5 mm
