File: Hardware/P2H-001.brd (EAGLE design)
At the start: 47 x 72 mm, 12 parts, among them K1 G5V1, T1 2SC1815, U1 ARDUINO_PRO_MINI

Commit message: New design.
Parts:
- removed D1, D2: BAS15, diode:DO34-7
- removed K1: G5V1, relay:G5V1
- removed OK1: 6N137, optocoupler:DIL08
- removed T1: 2SC1815, transistor:TO92-ECB
- removed U1: ARDUINO_PRO_MINI, SparkFun-Boards:ARDUINO_PRO_MINI
- added CN1: (no value), jst-ph:S4B-PH-K-S
- added IC1: 74LS07N, 74xx-us:DIL14
- added IC2: LTC485N, linear-technology:DIL08
- added JP2: (no value), pinhead:2X04
- added JP3: (no value), pinhead:1X04
- added JP4: (no value), pinhead:2X03
- added R4: 220, resistor:0204/5
- added U$1: ARDUINO_PRO_MINI, SparkFun-Boards:ARDUINO_PRO_MINI
- JP1: device pinhead:1X08 -> pinhead:1X05
- R2: value 3k -> 220
- R3: value 330 -> 120
- moved C1 53.4 mm to (10.2, 67.3), turned to 0 degrees
- moved JP1 44.7 mm to (41.9, 47.0)
- moved R3 43.4 mm to (36.8, 49.5)
- moved C2 42.2 mm to (27.9, 67.3), turned to 0 degrees
- moved R2 32.4 mm to (36.8, 34.3)
- moved R1 30.1 mm to (36.8, 41.9)
Connections:
- removed net MIDI0: JP1.3, R1.2
- removed net MIDI1: D1.A, JP1.4, OK1.3
- removed net RX: OK1.6, U1.2
- removed net VDD: C1.1, JP1.1, U1.24
- new net N$10: JP3.3, U$1.17
- new net N$11: JP3.4, U$1.9
- new net N$12: JP4.1, U$1.12
- new net N$14: JP4.3, U$1.7
- new net N$15: JP4.4, U$1.15
- new net N$16: JP4.5, U$1.14
- new net N$17: JP4.6, U$1.16
- new net N$18: CN1.1, IC2.6, R3.1
- new net N$19: CN1.2, IC2.7, R3.2
- new net N$7: JP1.5, R1.1
- new net N$9: JP2.1, JP2.3, U$1.24
- net GND: now also IC1.11, IC1.13, IC1.5, IC1.7, IC1.9, IC2.5, JP2.2, JP2.4, JP2.6, JP3.2, R4.2, U$1.23; no longer JP1.8, T1.E, U1.23
- net N$1: now also IC1.1, IC1.3, IC2.4, U$1.1; no longer JP1.5, K1.10
- net N$13: now also JP4.2, U$1.13; no longer D1.C, OK1.2, R1.1
- net N$2: now also IC1.2, R1.2; no longer D2.A, K1.9, T1.C
- net N$3: now also JP1.4; no longer U1.13
- net N$4: now also IC1.4, JP1.3; no longer R2.2, T1.B
- net N$5: now also JP2.8, R4.1; no longer JP1.6, K1.5
- net N$6: now also JP2.5, U$1.22; no longer R3.1, U1.16
- net N$8: now also JP2.7, U$1.6; no longer JP1.7, R3.2
- net VCC: now also C1.1, IC1.14, IC2.2, IC2.3, IC2.8, JP1.1, JP3.1, R2.2, U$1.21; no longer D2.C, K1.2, OK1.7, U1.21
Routing:
- net GND: track 73.3 -> 137.0 mm
- net VDD: track 62.6 -> 0.00 mm
- net MIDI1: track 46.5 -> 0.00 mm
- net N$15: track 0.00 -> 40.2 mm
- net N$6: track 64.9 -> 28.7 mm
- net N$17: track 0.00 -> 34.7 mm
- net N$16: track 0.00 -> 32.5 mm
- net N$10: track 0.00 -> 31.7 mm
- net N$9: track 0.00 -> 30.6 mm
- net VCC: track 76.7 -> 106.9 mm
- net N$4: track 7.62 -> 36.8 mm
- net N$3: track 46.6 -> 20.0 mm
- net N$1: track 30.4 -> 55.2 mm, vias 0 -> 1
- net RX: track 23.1 -> 0.00 mm
- net N$2: track 14.2 -> 37.3 mm
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Other:
- board text added: "PINEAPPLE II HYDROGEN REVISION 1.0.0 (2015)"
- board text removed: "P2H 0.0.0"
