File: Hardware/P2H-001.sch (EAGLE design)
At the start: 12 parts, among them K1 G5V1, T1 2SC1815, U1 ARDUINO_PRO_MINI

Commit message: New design.
Parts:
- removed D1, D2: BAS15, diode:BAS15
- removed K1: G5V1, relay:G5V1
- removed OK1: 6N137, optocoupler:6N137
- removed T1: 2SC1815, transistor:2SC1815
- added CN1: (no value), jst-ph:S4B-PH-K-S
- added IC1: 74LS07N, 74xx-us:74LS07N
- added IC2: LTC485N, linear-technology:LTC485N
- added JP2: (no value), pinhead:PINHD-2X4
- added JP3: (no value), pinhead:PINHD-1X4
- added JP4: (no value), pinhead:PINHD-2X3
- added R4: 220, resistor:R-US_0204/5
- JP1: device pinhead:PINHD-1X8 -> pinhead:PINHD-1X5
- R2: value 3k -> 220
- R3: value 330 -> 120
- renumbered U1 to U$1
Connections:
- removed net MIDI0: JP1.3, R1.2
- removed net MIDI1: D1.A, JP1.4, OK1.C
- removed net RX: OK1.VO, U$1.RXI
- removed net VDD: C1.1, JP1.1, U$1.RAW
- new net N$10: JP3.3, U$1.A0
- new net N$11: JP3.4, U$1.*6
- new net N$12: JP4.1, U$1.*9
- new net N$14: JP4.3, U$1.4
- new net N$15: JP4.4, U$1.12
- new net N$16: JP4.5, U$1.*11
- new net N$17: JP4.6, U$1.13
- new net N$18: CN1.1, IC2.A, R3.1
- new net N$19: CN1.2, IC2.B, R3.2
- new net N$7: JP1.5, R1.1
- new net N$9: JP2.1, JP2.3, U$1.RAW
- net GND: now also IC1C.I, IC1D.I, IC1E.I, IC1F.I, IC2.GND, JP2.2, JP2.4, JP2.6, JP3.2, R4.2; no longer JP1.8, T1.E
- net N$1: now also IC1A.I, IC1B.I, IC2.DI, U$1.TXO; no longer JP1.5, K12.S
- net N$13: now also JP4.2, U$1.*10; no longer D1.C, OK1.A, R1.1
- net N$2: now also IC1A.O, R1.2; no longer D2.A, K11.2, T1.C
- net N$3: now also JP1.4; no longer U$1.*10
- net N$4: now also IC1B.O, JP1.3; no longer R2.2, T1.B
- net N$5: now also JP2.8, R4.1; no longer JP1.6, K12.P
- net N$6: now also JP2.5, U$1.RST@2; no longer R3.1, U$1.13
- net N$8: now also JP2.7, U$1.*3; no longer JP1.7, R3.2
- net VCC: now also C1.1, IC2.!RE, IC2.DE, IC2.VCC, JP1.1, JP3.1, R2.2; no longer D2.C, K11.1, OK1.VE
Other:
- note removed: "1: Vdd 2: GND 3: MIDI RXA 4: MIDI RXK 5: RELAY COMMON 6: RELAY N.O. 7: LEDA 8: LEDK"
- moved on the sheet: R1, R2, R3
