File: Hardware/Board/P2H-001.brd (EAGLE design)
At the start: 45 x 45 mm, 15 parts, among them IC1 74LS07N, IC2 LTC485N

Commit message: Adopted new Hydroport pinout.
Connections:
- new net N$14: JP3.6, U$1.A5
- new net N$4: JP3.4, U$1.17
- net N$10: now also U$1.9; no longer U$1.A4
- net N$11: now also JP3.5, U$1.A4; no longer JP3.4, U$1.A5
Routing:
- net N$14: track 0.00 -> 28.5 mm
- net N$4: track 0.00 -> 15.5 mm
- net N$10: track 21.9 -> 17.8 mm
- net GND: track 151.1 -> 152.7 mm
Changed lines of the file:
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@@
 <contactref element="R5" pad="1"/>
 <contactref element="IC1" pad="3"/>
+<wire x1="40.005" y1="15.5448" x2="41.8338" y2="13.716" width="0.254" layer="1"/>
+<wire x1="40.005" y1="16.6878" x2="40.005" y2="15.5448" width="0.254" layer="1"/>
+<wire x1="41.8338" y1="18.5166" x2="40.005" y2="16.6878" width="0.254" layer="1"/>
+<wire x1="41.8338" y1="13.716" x2="42" y2="13.54" width="0.254" layer="1"/>
+<wire x1="41.8338" y1="18.5166" x2="42" y2="18.69" width="0.254" layer="1"/>
 <wire x1="23.5458" y1="4.3434" x2="21.2598" y2="4.3434" width="0.254" layer="1"/>
 <wire x1="21.2598" y1="4.3434" x2="21.23" y2="4.27" width="0.254" layer="1"/>
@@
 <wire x1="21.0312" y1="4.3434" x2="21.23" y2="4.27" width="0.254" layer="16"/>
 <wire x1="18.7452" y1="4.3434" x2="18.69" y2="4.27" width="0.254" layer="16"/>
+<wire x1="42.0624" y1="9.8298" x2="42.0624" y2="13.4874" width="0.254" layer="16"/>
+<wire x1="43.2054" y1="8.6868" x2="42.0624" y2="9.8298" width="0.254" layer="16"/>
+<wire x1="43.2054" y1="4.1148" x2="43.2054" y2="8.6868" width="0.254" layer="16"/>
+<wire x1="41.148" y1="2.0574" x2="43.2054" y2="4.1148" width="0.254" layer="16"/>
+<wire x1="36.1188" y1="2.0574" x2="41.148" y2="2.0574" width="0.254" layer="16"/>
+<wire x1="32.6898" y1="5.4864" x2="36.1188" y2="2.0574" width="0.254" layer="16"/>
+<wire x1="24.9174" y1="5.4864" x2="32.6898" y2="5.4864" width="0.254" layer="16"/>
+<wire x1="23.7744" y1="4.3434" x2="24.9174" y2="5.4864" width="0.254" layer="16"/>
+<wire x1="42.0624" y1="13.4874" x2="42" y2="13.54" width="0.254" layer="16"/>
+<wire x1="23.7744" y1="4.3434" x2="23.77" y2="4.27" width="0.254" layer="16"/>
 <wire x1="8.4582" y1="33.8328" x2="3.2004" y2="33.8328" width="0.254" layer="16"/>
 <wire x1="10.7442" y1="36.1188" x2="8.4582" y2="33.8328" width="0.254" layer="16"/>
@@
 <wire x1="41.8338" y1="35.433" x2="42" y2="35.27" width="0.254" layer="1"/>
 <wire x1="35.8902" y1="36.1188" x2="35.81" y2="36.31" width="0.254" layer="1"/>
-<wire x1="40.005" y1="15.5448" x2="41.8338" y2="13.716" width="0.254" layer="1"/>
-<wire x1="40.005" y1="16.6878" x2="40.005" y2="15.5448" width="0.254" layer="1"/>
-<wire x1="41.8338" y1="18.5166" x2="40.005" y2="16.6878" width="0.254" layer="1"/>
-<wire x1="41.8338" y1="13.716" x2="42" y2="13.54" width="0.254" layer="1"/>
-<wire x1="41.8338" y1="18.5166" x2="42" y2="18.69" width="0.254" layer="1"/>
 <wire x1="13.2588" y1="24.6888" x2="13.2588" y2="26.9748" width="0.254" layer="1"/>
 <wire x1="13.2588" y1="26.9748" x2="13.2588" y2="28.575" width="0.254" layer="1"/>
@@
 <wire x1="3.2004" y1="20.1168" x2="3" y2="19.96" width="0.254" layer="16"/>
 <wire x1="12.1158" y1="23.7744" x2="12.34" y2="23.62" width="0.254" layer="16"/>
-<wire x1="19.2024" y1="16.6878" x2="40.005" y2="16.6878" width="0.254" layer="1"/>
-<wire x1="12.3444" y1="23.5458" x2="19.2024" y2="16.6878" width="0.254" layer="1"/>
-<wire x1="12.3444" y1="23.5458" x2="12.34" y2="23.62" width="0.254" layer="1"/>
 <wire x1="35.2044" y1="36.1188" x2="35.6616" y2="36.1188" width="0.254" layer="1"/>
 <wire x1="33.6042" y1="34.5186" x2="35.2044" y2="36.1188" width="0.254" layer="1"/>
@@
 <wire x1="31.0896" y1="2.9718" x2="31.23" y2="3" width="0.254" layer="16"/>
 </signal>
-<signal name="N$10">
-<contactref element="JP3" pad="3"/>
-<contactref element="U$1" pad="A4"/>
-<wire x1="32.9184" y1="21.2598" x2="41.8338" y2="21.2598" width="0.254" layer="16"/>
-<wire x1="32.004" y1="22.1742" x2="32.9184" y2="21.2598" width="0.254" layer="16"/>
-<wire x1="22.6314" y1="22.1742" x2="32.004" y2="22.1742" width="0.254" layer="16"/>
-<wire x1="21.2598" y1="20.8026" x2="22.6314" y2="22.1742" width="0.254" layer="16"/>
-<wire x1="41.8338" y1="21.2598" x2="42" y2="21.23" width="0.254" layer="16"/>
-<wire x1="21.2598" y1="20.8026" x2="21.07125" y2="20.7625" width="0.254" layer="16"/>
-</signal>
-<signal name="N$11">
-<contactref element="U$1" pad="A5"/>
-<contactref element="JP3" pad="4"/>
-<wire x1="39.5478" y1="23.5458" x2="41.8338" y2="23.5458" width="0.254" layer="1"/>
-<wire x1="38.1762" y1="22.1742" x2="39.5478" y2="23.5458" width="0.254" layer="1"/>
-<wire x1="20.1168" y1="22.1742" x2="38.1762" y2="22.1742" width="0.254" layer="1"/>
-<wire x1="18.7452" y1="20.8026" x2="20.1168" y2="22.1742" width="0.254" layer="1"/>
-<wire x1="41.8338" y1="23.5458" x2="42" y2="23.77" width="0.254" layer="1"/>
-<wire x1="18.7452" y1="20.8026" x2="18.53125" y2="20.7625" width="0.254" layer="1"/>
-</signal>
 <signal name="N$2">
 <contactref element="R1" pad="2"/>
@@
 <wire x1="14.859" y1="41.8338" x2="15.04" y2="42" width="0.254" layer="1"/>
 </signal>
+<signal name="N$4">
+<contactref element="U$1" pad="17"/>
+<contactref element="JP3" pad="4"/>
+<wire x1="39.5478" y1="23.7744" x2="41.8338" y2="23.7744" width="0.254" layer="1"/>
+<wire x1="38.4048" y1="24.9174" x2="39.5478" y2="23.7744" width="0.254" layer="1"/>
+<wire x1="28.8036" y1="24.9174" x2="38.4048" y2="24.9174" width="0.254" layer="1"/>
+<wire x1="27.6606" y1="23.7744" x2="28.8036" y2="24.9174" width="0.254" layer="1"/>
+<wire x1="41.8338" y1="23.7744" x2="42" y2="23.77" width="0.254" layer="1"/>
+<wire x1="27.6606" y1="23.7744" x2="27.58" y2="23.62" width="0.254" layer="1"/>
+</signal>
+<signal name="N$10">
+<contactref element="U$1" pad="9"/>
+<contactref element="JP3" pad="3"/>
+<wire x1="30.1752" y1="9.3726" x2="41.8338" y2="21.0312" width="0.254" layer="1"/>
+<wire x1="30.1752" y1="8.4582" x2="30.1752" y2="9.3726" width="0.254" layer="1"/>
+<wire x1="41.8338" y1="21.0312" x2="42" y2="21.23" width="0.254" layer="1"/>
+<wire x1="30.1752" y1="8.4582" x2="30.12" y2="8.38" width="0.254" layer="1"/>
+</signal>
+<signal name="N$11">
+<contactref element="U$1" pad="A4"/>
+<contactref element="JP3" pad="5"/>
+<wire x1="39.5478" y1="24.003" x2="41.8338" y2="26.289" width="0.254" layer="16"/>
+<wire x1="39.5478" y1="22.86" x2="39.5478" y2="24.003" width="0.254" layer="16"/>
+<wire x1="36.1188" y1="19.431" x2="39.5478" y2="22.86" width="0.254" layer="16"/>
+<wire x1="22.4028" y1="19.431" x2="36.1188" y2="19.431" width="0.254" layer="16"/>
+<wire x1="21.2598" y1="20.574" x2="22.4028" y2="19.431" width="0.254" layer="16"/>
+<wire x1="41.8338" y1="26.289" x2="42" y2="26.31" width="0.254" layer="16"/>
+<wire x1="21.2598" y1="20.574" x2="21.07125" y2="20.7625" width="0.254" layer="16"/>
+</signal>
+<signal name="N$14">
+<contactref element="U$1" pad="A5"/>
+<contactref element="JP3" pad="6"/>
+<wire x1="39.0906" y1="26.0604" x2="41.8338" y2="28.8036" width="0.254" layer="16"/>
+<wire x1="39.0906" y1="23.0886" x2="39.0906" y2="26.0604" width="0.254" layer="16"/>
+<wire x1="38.1762" y1="22.1742" x2="39.0906" y2="23.0886" width="0.254" layer="16"/>
+<wire x1="20.1168" y1="22.1742" x2="38.1762" y2="22.1742" width="0.254" layer="16"/>
+<wire x1="18.7452" y1="20.8026" x2="20.1168" y2="22.1742" width="0.254" layer="16"/>
+<wire x1="41.8338" y1="28.8036" x2="42" y2="28.85" width="0.254" layer="16"/>
+<wire x1="18.7452" y1="20.8026" x2="18.53125" y2="20.7625" width="0.254" layer="16"/>
+</signal>
 </signals>

Commit message: Changed layout of ZeroVoltage.
Parts:
- R2: value 220 -> 330
- R3: value 120 -> 220
- R4: value 220 -> 120
- R5: value 330 -> 150
- moved R3 41.7 mm to (3.00, 12.5), turned to 90 degrees
- moved R4 32.4 mm to (32.5, 42.0), turned to 0 degrees
- moved R5 30.6 mm to (42.0, 11.0), turned to 90 degrees
- moved R2 13.4 mm to (12.5, 3.00), turned to 0 degrees
Connections:
- net GND: now also R2.1, R5.2; no longer R4.2, R5.1
- net N$13: now also R2.2; no longer R5.2
- net N$18: now also R4.1; no longer R3.1
- net N$19: now also R4.2; no longer R3.2
- net N$3: now also R3.1; no longer R2.1
- net N$5: now also R5.1; no longer R4.1
- net VCC: now also R3.2; no longer R2.2
Changed lines of the file:
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@@
 <element name="JP1" library="pinhead" package="1X05" value="" x="3" y="22.5" rot="R90"/>
 <element name="IC1" library="74xx-us" package="DIL14" value="74LS07N" x="16" y="32.5"/>
-<element name="R2" library="resistor" package="0204/5" value="220" x="3" y="12.5" rot="R90"/>
+<element name="R3" library="resistor" package="0204/5" value="220" x="3" y="12.5" rot="R90"/>
 <element name="JP2" library="pinhead" package="2X04" value="" x="22.5" y="3"/>
-<element name="R4" library="resistor" package="0204/5" value="220" x="42" y="11" rot="R90"/>
+<element name="R5" library="resistor" package="0204/5" value="150" x="42" y="11" rot="R90"/>
 <element name="JP3" library="pinhead" package="1X06" value="" x="42" y="22.5" rot="R90"/>
 <element name="IC2" library="linear-technology" package="DIL08" value="LTC485N" x="32" y="32.5">
@@
 <attribute name="OC_FARNELL" value="unknown" x="32" y="32.5" size="1.778" layer="27" display="off"/>
 </element>
-<element name="R3" library="resistor" package="0204/5" value="120" x="32.5" y="42"/>
+<element name="R4" library="resistor" package="0204/5" value="120" x="32.5" y="42"/>
 <element name="CN1" library="jst-ph" package="B4B-PH-K-S" value="" x="22.5" y="42"/>
+<element name="R2" library="resistor" package="0204/5" value="330" x="12.5" y="3"/>
+<element name="LED1" library="led" package="LED3MM" value="" x="32.5" y="3" rot="R180"/>
 <element name="U$1" library="SparkFun-Boards" package="ARDUINO_PRO_MINI" value="ARDUINO_PRO_MINI" x="22.5" y="16" rot="R90"/>
-<element name="R5" library="resistor" package="0204/5" value="330" x="12.5" y="3"/>
-<element name="LED1" library="led" package="LED3MM" value="" x="32.5" y="3" rot="R180"/>
 </elements>
 <signals>
@@
 <contactref element="JP2" pad="4"/>
 <contactref element="JP2" pad="6"/>
-<contactref element="R4" pad="2"/>
+<contactref element="R5" pad="2"/>
 <contactref element="JP3" pad="2"/>
 <contactref element="IC2" pad="5"/>
@@
 <contactref element="IC1" pad="11"/>
 <contactref element="IC1" pad="9"/>
+<contactref element="R2" pad="1"/>
+<contactref element="IC1" pad="3"/>
 <contactref element="U$1" pad="23"/>
-<contactref element="R5" pad="1"/>
-<contactref element="IC1" pad="3"/>
 <wire x1="40.005" y1="15.5448" x2="41.8338" y2="13.716" width="0.254" layer="1"/>
 <wire x1="40.005" y1="16.6878" x2="40.005" y2="15.5448" width="0.254" layer="1"/>
@@
 <contactref element="IC2" pad="3"/>
 <contactref element="IC2" pad="2"/>
-<contactref element="R2" pad="2"/>
+<contactref element="R3" pad="2"/>
 <contactref element="IC2" pad="8"/>
 <contactref element="C1" pad="1"/>
@@
 <signal name="N$1">
 <contactref element="IC2" pad="4"/>
+<contactref element="IC1" pad="1"/>
 <contactref element="U$1" pad="1"/>
-<contactref element="IC1" pad="1"/>
 <wire x1="8.4582" y1="23.0886" x2="8.4582" y2="28.575" width="0.254" layer="1"/>
 <wire x1="11.6586" y1="19.8882" x2="8.4582" y2="23.0886" width="0.254" layer="1"/>
@@
 </signal>
 <signal name="N$3">
-<contactref element="R2" pad="1"/>
+<contactref element="R3" pad="1"/>
 <contactref element="JP1" pad="4"/>
 <wire x1="2.9718" y1="13.4874" x2="2.9718" y2="10.0584" width="0.254" layer="1"/>
@@
 </signal>
 <signal name="N$5">
-<contactref element="R4" pad="1"/>
+<contactref element="R5" pad="1"/>
 <contactref element="JP2" pad="8"/>
 <wire x1="42.0624" y1="6.858" x2="42.0624" y2="8.4582" width="0.254" layer="1"/>
@@
 <signal name="N$18">
 <contactref element="IC2" pad="6"/>
-<contactref element="R3" pad="1"/>
+<contactref element="R4" pad="1"/>
 <contactref element="CN1" pad="1"/>
 <wire x1="20.1168" y1="41.8338" x2="19.6596" y2="41.8338" width="0.254" layer="16"/>
@@
 </signal>
 <signal name="N$19">
-<contactref element="R3" pad="2"/>
+<contactref element="R4" pad="2"/>
 <contactref element="IC2" pad="7"/>
 <contactref element="CN1" pad="2"/>
@@
 </signal>
 <signal name="N$12">
+<contactref element="LED1" pad="A"/>
 <contactref element="U$1" pad="8"/>
-<contactref element="LED1" pad="A"/>
 <wire x1="32.6898" y1="3.2004" x2="33.6042" y2="3.2004" width="0.254" layer="1"/>
 <wire x1="27.6606" y1="8.2296" x2="32.6898" y2="3.2004" width="0.254" layer="1"/>
@@
 <signal name="N$13">
 <contactref element="LED1" pad="K"/>
-<contactref element="R5" pad="2"/>
+<contactref element="R2" pad="2"/>
 <wire x1="31.0896" y1="2.9718" x2="15.0876" y2="2.9718" width="0.254" layer="16"/>
 <wire x1="15.0876" y1="2.9718" x2="15.04" y2="3" width="0.254" layer="16"/>
@@
 </signal>
 <signal name="N$4">
+<contactref element="JP3" pad="4"/>
 <contactref element="U$1" pad="17"/>
-<contactref element="JP3" pad="4"/>
 <wire x1="39.5478" y1="23.7744" x2="41.8338" y2="23.7744" width="0.254" layer="1"/>
 <wire x1="38.4048" y1="24.9174" x2="39.5478" y2="23.7744" width="0.254" layer="1"/>
@@
 </signal>
 <signal name="N$10">
+<contactref element="JP3" pad="3"/>
 <contactref element="U$1" pad="9"/>
-<contactref element="JP3" pad="3"/>
 <wire x1="30.1752" y1="9.3726" x2="41.8338" y2="21.0312" width="0.254" layer="1"/>
 <wire x1="30.1752" y1="8.4582" x2="30.1752" y2="9.3726" width="0.254" layer="1"/>
@@
 </signal>
 <signal name="N$11">
+<contactref element="JP3" pad="5"/>
 <contactref element="U$1" pad="A4"/>
-<contactref element="JP3" pad="5"/>
 <wire x1="39.5478" y1="24.003" x2="41.8338" y2="26.289" width="0.254" layer="16"/>
 <wire x1="39.5478" y1="22.86" x2="39.5478" y2="24.003" width="0.254" layer="16"/>
@@
 </signal>
 <signal name="N$14">
+<contactref element="JP3" pad="6"/>
 <contactref element="U$1" pad="A5"/>
-<contactref element="JP3" pad="6"/>
 <wire x1="39.0906" y1="26.0604" x2="41.8338" y2="28.8036" width="0.254" layer="16"/>
 <wire x1="39.0906" y1="23.0886" x2="39.0906" y2="26.0604" width="0.254" layer="16"/>

Commit message: Clean up.
Parts:
- moved R5 27.3 mm to (33.0, 36.8), turned to 0 degrees
- moved R3 26.2 mm to (12.7, 36.8), turned to 0 degrees
- moved R4 2.68 mm to (33.0, 39.4)
- moved R1 2.64 mm to (12.7, 39.4)
- moved IC2 2.26 mm to (33.0, 30.5)
- moved IC1 2.08 mm to (16.5, 30.5)
- moved C2 1.68 mm to (40.6, 33.0)
- moved C1 0.96 mm to (3.81, 33.0)
- moved LED1 0.96 mm to (33.0, 3.81)
- moved U$1 0.84 mm to (22.9, 15.2)
- moved R2 0.83 mm to (12.7, 3.81)
Routing:
- net N$5: track 23.3 -> 45.9 mm, vias 0 -> 2
- net VCC: track 109.8 -> 91.7 mm
- net N$6: track 36.8 -> 32.0 mm
- net N$9: track 31.8 -> 28.5 mm
- net GND: track 152.7 -> 150.1 mm, vias 0 -> 1
- net N$1: track 51.3 -> 48.7 mm
- net N$7: track 17.3 -> 14.8 mm
- net N$11: track 25.0 -> 27.2 mm
- net N$3: track 16.6 -> 14.8 mm
- net N$19: track 19.1 -> 20.4 mm
- net N$13: track 16.2 -> 17.2 mm
- net N$14: track 28.5 -> 27.6 mm, vias 0 -> 1
- net N$8: track 8.22 -> 7.31 mm
- net N$2: track 15.0 -> 14.3 mm
- net N$4: track 15.5 -> 14.8 mm
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