File: Hardware/Board/P2D-001.sch (EAGLE design)
At the start: 21 parts, among them IC1 LTC485N, K1 G5V1, T1 2SC1815

Commit message: Overhaul.
Connections:
- net GND: now also JP2.3; no longer JP2.2
- net N$10: now also JP2.4, U$1.*5; no longer JP2.1, R1.1
- net N$18: now also JP2.1, K12.P@1; no longer JP2.3, K12.P
- net N$19: now also JP2.2; no longer JP2.4
- net VCC: no longer R1.2
Other:
- note added: "HYDROGEN CONNECTOR (h) 1,3: Power; 2, 4: GND; 5-6: Reset; 7-8: LED"
- note added: "MIDIIN (m1) 1: NC; 2: NC; 3: NC; 4: MIDI IN Anode; 5: MIDI IN Kathode"
- note added: "MIDISTANCE (c) 1: NC 2: NC; 3: RX+; 4: RX-"
- note added: "Pineapple II Deuterium 1.0.0 Copyright 2015 by Pineapple.cc"
- note added: "ZEROVOLT DRIVE (z) 1: CONTACT A; 2: CONTACT B; 3: GND; 4: GPIO"
- note removed: "1,3: Power; 2, 4: GND; 5-6: Reset; 7-8: LED"
- note removed: "1: Power; 2: GND; 3: Raw TX; 4: MIDI IN Anode; 5: MIDI IN Kathode"
- note removed: "1: TX+; 2: TX-; 3: RX+; 4: RX-"
- note removed: "Pineapple II Hydrogen 2 0.0.0 Copyright 2015 by Pineapple.cc"
- moved on the sheet: R1
Changed lines of the file:
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@@
 <part name="JP2" library="pinhead" deviceset="PINHD-1X4" device=""/>
 <part name="SUPPLY2" library="supply2" deviceset="GND" device=""/>
-<part name="SUPPLY1" library="supply2" deviceset="VCC" device=""/>
 <part name="R6" library="resistor" deviceset="R-US_" device="0204/5" value="120"/>
 <part name="IC1" library="linear-technology" deviceset="LTC485" device="N"/>
@@
 <sheet>
 <plain>
-<text x="12.7" y="-15.24" size="1.778" layer="91">Pineapple II Hydrogen 2 0.0.0
+<text x="12.7" y="-15.24" size="1.778" layer="91">Pineapple II Deuterium 1.0.0
 Copyright 2015 by Pineapple.cc</text>
-<text x="152.4" y="60.96" size="1.778" layer="91">1: TX+; 2: TX-;
+<text x="152.4" y="60.96" size="1.778" layer="91">MIDISTANCE (c)
+1: NC 2: NC;
 3: RX+; 4: RX-</text>
-<text x="10.16" y="88.9" size="1.778" layer="91">1: Power; 2: GND; 3: Raw TX;
+<text x="10.16" y="86.36" size="1.778" layer="91">MIDIIN (m1)
+1: NC; 2: NC; 3: NC;
 4: MIDI IN Anode; 5: MIDI IN Kathode</text>
-<text x="93.98" y="25.4" size="1.778" layer="91">1,3: Power; 2, 4: GND;
+<text x="127" y="38.1" size="1.778" layer="91">HYDROGEN CONNECTOR (h)
+1,3: Power; 2, 4: GND;
 5-6: Reset;
 7-8: LED</text>
+<text x="48.26" y="-7.62" size="1.778" layer="91">ZEROVOLT DRIVE (z)
+1: CONTACT A; 2: CONTACT B;
+3: GND; 4: GPIO</text>
 </plain>
 <instances>
@@
 <instance part="SUPPLY9" gate="GND" x="121.92" y="33.02"/>
 <instance part="R5" gate="G$1" x="114.3" y="38.1"/>
-<instance part="R1" gate="G$1" x="27.94" y="17.78" rot="R90"/>
+<instance part="R1" gate="G$1" x="12.7" y="58.42" rot="R90"/>
 <instance part="CN1" gate="G$1" x="157.48" y="78.74"/>
 <instance part="R4" gate="G$1" x="106.68" y="12.7" rot="R90"/>
@@
 <instance part="R3" gate="G$1" x="45.72" y="30.48"/>
 <instance part="JP2" gate="A" x="35.56" y="5.08"/>
-<instance part="SUPPLY2" gate="GND" x="27.94" y="-2.54"/>
-<instance part="SUPPLY1" gate="G$1" x="27.94" y="27.94"/>
+<instance part="SUPPLY2" gate="GND" x="20.32" y="-2.54"/>
 <instance part="R6" gate="G$1" x="144.78" y="76.2"/>
 <instance part="IC1" gate="G$1" x="119.38" y="76.2"/>
@@
 <pinref part="SUPPLY8" gate="GND" pin="GND"/>
 <wire x1="106.68" y1="5.08" x2="106.68" y2="7.62" width="0.1524" layer="91"/>
-</segment>
-<segment>
-<pinref part="JP2" gate="A" pin="2"/>
-<pinref part="SUPPLY2" gate="GND" pin="GND"/>
-<wire x1="33.02" y1="7.62" x2="27.94" y2="7.62" width="0.1524" layer="91"/>
-<wire x1="27.94" y1="7.62" x2="27.94" y2="0" width="0.1524" layer="91"/>
 </segment>
 <segment>
@@
 <junction x="132.08" y="66.04"/>
 </segment>
+<segment>
+<pinref part="JP2" gate="A" pin="3"/>
+<pinref part="SUPPLY2" gate="GND" pin="GND"/>
+<wire x1="33.02" y1="5.08" x2="20.32" y2="5.08" width="0.1524" layer="91"/>
+<wire x1="20.32" y1="5.08" x2="20.32" y2="0" width="0.1524" layer="91"/>
+</segment>
 </net>
 <net name="VCC" class="0">
@@
 <wire x1="40.64" y1="53.34" x2="33.02" y2="53.34" width="0.1524" layer="91"/>
 <junction x="33.02" y="53.34"/>
-</segment>
-<segment>
-<pinref part="SUPPLY1" gate="G$1" pin="VCC"/>
-<wire x1="27.94" y1="25.4" x2="27.94" y2="22.86" width="0.1524" layer="91"/>
-<pinref part="R1" gate="G$1" pin="2"/>
 </segment>
 </net>
@@
 </segment>
 </net>
-<net name="N$18" class="0">
-<segment>
-<pinref part="K1" gate="2" pin="P"/>
-<wire x1="22.86" y1="5.08" x2="22.86" y2="40.64" width="0.1524" layer="91"/>
-<pinref part="JP2" gate="A" pin="3"/>
-<wire x1="33.02" y1="5.08" x2="22.86" y2="5.08" width="0.1524" layer="91"/>
-</segment>
-</net>
 <net name="N$19" class="0">
 <segment>
 <pinref part="K1" gate="2" pin="S"/>
 <wire x1="17.78" y1="48.26" x2="15.24" y2="48.26" width="0.1524" layer="91"/>
-<wire x1="15.24" y1="48.26" x2="15.24" y2="2.54" width="0.1524" layer="91"/>
-<pinref part="JP2" gate="A" pin="4"/>
-<wire x1="33.02" y1="2.54" x2="15.24" y2="2.54" width="0.1524" layer="91"/>
+<wire x1="15.24" y1="48.26" x2="15.24" y2="7.62" width="0.1524" layer="91"/>
+<pinref part="JP2" gate="A" pin="2"/>
+<wire x1="15.24" y1="7.62" x2="33.02" y2="7.62" width="0.1524" layer="91"/>
 </segment>
 </net>
@@
 <pinref part="R3" gate="G$1" pin="1"/>
 <wire x1="40.64" y1="30.48" x2="38.1" y2="30.48" width="0.1524" layer="91"/>
-</segment>
-</net>
-<net name="N$10" class="0">
-<segment>
-<wire x1="27.94" y1="12.7" x2="27.94" y2="10.16" width="0.1524" layer="91"/>
-<pinref part="JP2" gate="A" pin="1"/>
-<wire x1="27.94" y1="10.16" x2="33.02" y2="10.16" width="0.1524" layer="91"/>
-<pinref part="R1" gate="G$1" pin="1"/>
 </segment>
 </net>
@@
 </segment>
 </net>
+<net name="N$18" class="0">
+<segment>
+<pinref part="K1" gate="2" pin="P@1"/>
+<wire x1="20.32" y1="40.64" x2="20.32" y2="10.16" width="0.1524" layer="91"/>
+<pinref part="JP2" gate="A" pin="1"/>
+<wire x1="20.32" y1="10.16" x2="33.02" y2="10.16" width="0.1524" layer="91"/>
+</segment>
+</net>
+<net name="N$10" class="0">
+<segment>
+<pinref part="U$1" gate="G$1" pin="*5"/>
+<wire x1="60.96" y1="27.94" x2="38.1" y2="27.94" width="0.1524" layer="91"/>
+<wire x1="38.1" y1="27.94" x2="38.1" y2="15.24" width="0.1524" layer="91"/>
+<wire x1="38.1" y1="15.24" x2="27.94" y2="15.24" width="0.1524" layer="91"/>
+<wire x1="27.94" y1="15.24" x2="27.94" y2="2.54" width="0.1524" layer="91"/>
+<pinref part="JP2" gate="A" pin="4"/>
+<wire x1="27.94" y1="2.54" x2="33.02" y2="2.54" width="0.1524" layer="91"/>
+</segment>
+</net>
